Commit message: urdf edited and rtabmap launch file, config edited.

File: minibot_ws/src/minibot_description/urdf/minibot.urdf (robot description, URDF)
Before this commit: robot minibot, 21 links, 20 joints
Links:
- link zed_camera_center: geometry collision mesh filename=file:///opt/ros/humble/share/zed_description/meshes/zed2i.s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; visual mesh filename=file:///opt/ros/humble/share/zed_description/meshes/zed2i.s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
Joints:
- joint zed_camera_center_joint: origin xyz=0 0 0.015 rpy=0 0.0 0 -> xyz=0 0 0.016 rpy=0 0.0 0
- joint zed_mount_joint: origin xyz=0.12 0 0.425 rpy=0 0 0 -> xyz=0.19 0 0.410 rpy=0 0 0
